File: hardware/kicad/WeatherStation/communication.kicad_sch (KiCad schematic)
At the start: 10 parts, among them J6 SMA_Female_Edge, J7 DEBUG UART, U8 SX1276

Commit message: fix: remove invalid ;; comments from KiCad schematics and add SD card circuit
KiCad's S-expression parser does not support semicolon comments.
All ;; comment lines have been stripped from the 5 .kicad_sch files
and WeatherStation.kicad_sym to fix "Expecting '('" parse errors.

Also adds the SD card circuit to communication.kicad_sch:
- J22 MicroSD_SPI holder with SPI2 bus connections
- C38 100nF VCC decoupling capacitor
- R27 10k pull-up on card detect line
- SPI2_SCK/MISO/MOSI/SD_CS/SD_DET hierarchical labels
- Wire routing and power symbols (+3V3, GND)

https://claude.ai/code/session_01XHnfZQ5BbxTCTBMCteQyVe
Parts:
- added C38: 100nF, Capacitor_SMD:C_0402_1005Metric, symbol Device:C
- added J22: MicroSD_SPI, Connector:MicroSD_Molex_5031821852, symbol WeatherStation:MicroSD_SPI
- added R27: 10k, Resistor_SMD:R_0402_1005Metric, symbol Device:R
Connections:
- net GND is gone; now on net +3V3: C10.2 (-), C11.2, C12.2, C13.2, J6.2 (GND), J7.4 (Pin_4), U8.10 (GND), U8.29 (GND_PAD)
Other:
- note added: "SD CARD (SPI2 shared bus) Micro-SD holder (Molex 5031821852) CS=PD10, DET=PD11 (active low) Shared with W5500 Ethernet (CS=PB12)"

Commit message: feat: add ATWINC1500, RN4870, W5500, SIM7600 to communication schematic
Add all 4 industrial communication module circuits to communication.kicad_sch:

- U12 ATWINC1500 WiFi (SPI3): QFN-28, J18 SMA antenna, C28/C29 decoupling
- U13 RN4870 BLE (USART3): UART module, C30/C31 decoupling
- U14 W5500 Ethernet (SPI2): LQFP-48, Y2 25MHz crystal + C32/C33 load caps,
  J19 RJ45 Magjack, C26/C34 decoupling
- U15 SIM7600E-H Cellular (UART4): LTE Cat-4, U16 TPS7A2033 3.8V LDO,
  C36/C37 bulk caps (100uF+470uF), J20 Nano-SIM, J21 LTE SMA antenna

Also adds lib_symbols for all new components (ATWINC1500, RN4870, W5500,
SIM7600EH, TPS7A2033, RJ45_Magjack, NanoSIM_Holder, Crystal), updates
paper size to A2, and replaces ESP32 references with STM32 pin assignments.

https://claude.ai/code/session_01XHnfZQ5BbxTCTBMCteQyVe
Parts:
- added C26, C29: 10uF, Capacitor_SMD:C_0805_2012Metric, symbol Device:C_Polarized
- added C28, C30, C34: 100nF, Capacitor_SMD:C_0402_1005Metric, symbol Device:C
- added C31: 4.7uF, Capacitor_SMD:C_0805_2012Metric, symbol Device:C_Polarized
- added C32, C33: 18pF, Capacitor_SMD:C_0402_1005Metric, symbol Device:C
- added C35: 1uF, Capacitor_SMD:C_0402_1005Metric, symbol Device:C
- added C36: 100uF, Capacitor_SMD:CP_Elec_6.3x7.7, symbol Device:C_Polarized
- added C37: 470uF, Capacitor_SMD:CP_Elec_8x10.5, symbol Device:C_Polarized
- added J18: SMA_WiFi, Connector_Coaxial:SMA_Amphenol_132289_EdgeMount, symbol WeatherStation:SMA_Edge_Mount
- added J19: RJ45_Magjack, Connector_RJ:RJ45_Amphenol_ARJM11C7, symbol WeatherStation:RJ45_Magjack
- added J20: Nano-SIM, Connector:NanoSIM_Molex_78800-0001, symbol WeatherStation:NanoSIM_Holder
- added J21: SMA_LTE, Connector_Coaxial:SMA_Amphenol_132289_EdgeMount, symbol WeatherStation:SMA_Edge_Mount
- added U12: ATWINC1500-MR210PB, Package_DFN_QFN:QFN-28-1EP_5x5mm_P0.5mm_EP3.1x3.1mm, symbol WeatherStation:ATWINC1500
- added U13: RN4870-I/RM, WeatherStation:RN4870_11.5x8mm, symbol WeatherStation:RN4870
- added U14: W5500, Package_QFP:LQFP-48_7x7mm_P0.5mm, symbol WeatherStation:W5500
- added U15: SIM7600E-H, WeatherStation:SIM7600EH_LCC, symbol WeatherStation:SIM7600EH
- added U16: TPS7A2033 (3.8V), Package_TO_SOT_SMD:SOT-23-5, symbol WeatherStation:TPS7A2033
- added Y2: 25MHz, Crystal:Crystal_SMD_ABM3B_5x3.2mm, symbol Device:Crystal
Connections:
- net +3V3: now also C26.1 (+), C26.2 (-), C28.1, C28.2, C29.1 (+), C29.2 (-), C30.1, C30.2, C31.1 (+), C31.2 (-), C32.2, C33.2, C34.1, C34.2, C35.2, C36.1 (+), C36.2 (-), C37.1 (+), C37.2 (-), J18.2 (GND), J19.9 (SHIELD), J20.C5 (GND), J21.2 (GND), U12.29 (GND_PAD), U12.8 (VCC), U12.9 (GND), U13.5 (VCC), U13.6 (GND), U14.7 (VCC), U14.8 (GND), U15.7 (VBAT), U15.8 (GND), U16.2 (GND), U16.3 (EN)
- new net: C32.1, Y2.1
- new net: C33.1, J19.3 (RX+), J19.6 (RX-), U14.15 (LINKLED), Y2.2
- new net: J18.1 (Signal), U12.10 (ANT)
- new net: J21.1 (Signal), U15.9 (ANT_MAIN)
- new net BLE_RST: U13.3 (RST)
- new net BLE_STATUS: U13.4 (STATUS)
- new net BLE_TX: U13.1 (TX)
- new net CELL_DTR: U15.5 (DTR)
- new net CELL_PWRKEY: U15.3 (PWRKEY)
- new net CELL_RI: U15.6 (RI)
- new net CELL_RX: U15.2 (TXD)
- new net CELL_STATUS: U15.4 (STATUS)
- new net CELL_TX: U15.1 (RXD)
- new net SPI3_MISO: U12.2 (MISO)
- new net SPI3_MOSI: U12.3 (MOSI)
- new net SPI3_SCK: U12.1 (SCK)
- new net WIFI_CS: U12.4 (SSn)
- new net WIFI_EN: U12.7 (CHIP_EN)
- new net WIFI_IRQ: U12.6 (IRQn)
- new net WIFI_RST: U12.5 (RESETn)
Other:
- note added: "ATWINC1500 WiFi (SPI3): PE3 CS, PE4 RST, PE5 IRQ, PE6 EN RN4870 BLE (USART3): PB10 TX, PB11 RX, PD8 RST, PD9 STATUS W5500 Ethernet (SPI2): PB12 CS, PD3 RST, PD4 INT SIM7600E-H Cellular (UART4): PC10 TX, PC11 RX"
- note added: "ATWINC1500 WiFi Module (SPI3) IEEE 802.11 b/g/n, QFN-28 SPI3: PB3 SCK, PB4 MISO, PB5 MOSI CS=PE3, RST=PE4, IRQ=PE5, EN=PE6"
- note added: "All modules operate on 3.3V except SIM7600 which requires 3.4-4.2V via TPS7A2033 LDO"
- note added: "Industrial Communication Modules"
- note added: "RN4870 BLE Module (USART3) Bluetooth 5.0 Low Energy TX=PB10, RX=PB11 RST=PD8, STATUS=PD9"
- note added: "SIM7600E-H 4G/LTE Cellular Module (UART4) PC10 TX, PC11 RX, PD5 PWRKEY PD6 STATUS, PD7 DTR, PE2 RI Powered by TPS7A2033 3.8V LDO VBAT: 3.4-4.2V, 2A burst current"
- note added: "SPI1 Interface (LoRa): MOSI = PA7 MISO = PA6 SCK = PA5 NSS = PA4 (Chip Select) Reset = PC4 DIO0 (IRQ) = PC5"
- note added: "W5500 Ethernet Controller (SPI2) Hardwired TCP/IP, LQFP-48 SPI2: PB13 SCK, PB14 MISO, PB15 MOSI CS=PB12, RST=PD3, INT=PD4 25MHz crystal + RJ45 with magnetics"
- note removed: "KEEP-OUT ZONE 10mm x 10mm No copper/components in antenna keep-out zone"
- note removed: "SPI Interface: MOSI = GPIO10 MISO = GPIO11 SCK = GPIO12 NSS = GPIO13 (Chip Select) Reset = GPIO14 DIO0 (IRQ) = GPIO15"
- note removed: "Using ESP32-S3-WROOM-1 onboard PCB antenna. ANTENNA KEEP-OUT ZONE: 10mm x 10mm No copper pour, traces, or components in antenna keep-out zone. Keep-out extends beyond module edge on PCB. See module datasheet for exact dimensions and placement."
- note removed: "WiFi/BLE Antenna (ESP32-S3-WROOM-1)"
