File: hardware/kicad/WeatherStation/WeatherStation.kicad_sch (KiCad schematic)
At the start: 9 parts, among them SW1 BOOT, SW2 RESET, U1 ESP32-S3-WROOM-1-N16R8I

Commit message: Update KiCad schematic with detailed sensor interface design
Expanded the top-level schematic with comprehensive sensor interfaces
including I2C, SPI, UART, and ADC connections for the ESP32-S3 weather
station. Added hierarchical design structure with proper pin assignments.

https://claude.ai/code/session_01XHnfZQ5BbxTCTBMCteQyVe
Parts:
- removed C1: 10uF, symbol Device:C
- removed D6: Green, symbol Device:LED
- removed R4: 10k, symbol Device:R
- removed R5: 330R, symbol Device:R
- removed U1: ESP32-S3-WROOM-1-N16R8I, symbol WeatherStation:ESP32-S3-WROOM-1
- added C1: 10uF, Capacitor_SMD:C_0805_2012Metric, symbol Device:C_Polarized
- added D1: LED_GREEN, LED_SMD:LED_0603_1608Metric, symbol Device:LED
- added R1, R2: 10K, Resistor_SMD:R_0402_1005Metric, symbol Device:R
- added U1: ESP32-S3-WROOM-1, RF_Module:ESP32-S3-WROOM-1, symbol RF_Module:ESP32-S3-WROOM-1
- C2: footprint (none) -> Capacitor_SMD:C_0402_1005Metric
- R3: value 10k -> 330R; footprint (none) -> Resistor_SMD:R_0402_1005Metric
- SW1: value BOOT -> RESET; footprint (none) -> Button_Switch_SMD:SW_SPST_TL3342
- SW2: value RESET -> BOOT; footprint (none) -> Button_Switch_SMD:SW_SPST_TL3342
Connections:
- net GND: now also SW1.1, SW2.2
- net at SW2.1: now also R2.2
- net at SW1.2: now also R1.2
Other:
- sheet Communication ports: added none; removed +3V3, GND, LORA_CS, LORA_DIO0, LORA_RST, SPI_SCK
- sheet Industry Modules ports: added DEEP_SOIL, LEAF_WETNESS, SOIL_MOISTURE_ADC, SOIL_TEMP; removed +3V3, DEEP_SOIL_ADC, GND, INDUSTRY_ADC, LEAF_WET_ADC, ONEWIRE_A, ONEWIRE_B, POWER_PULSE
- sheet Power Supply ports: added VBATT, VSOLAR; removed +5V, +VBAT, BATT_SENSE
- sheet Sensors ports: added BATT_ADC, RAIN_GAUGE_INT, SCL, SDA, SPI_MOSI, WIND_SPEED_INT; removed +3V3, GND, I2C_SCL, I2C_SDA, RAIN_GAUGE, WIND_SPEED
- note added: "ESP32-S3 Weather Station - Top Level Schematic"
- note added: "Pin Assignments: I2C: GPIO8(SDA), GPIO9(SCL) SPI: GPIO10(MOSI), GPIO11(MISO), GPIO12(SCK), GPIO13(CS), GPIO14(RST), GPIO15(DIO0) Interrupts: GPIO4(Wind), GPIO5(Rain) ADC: GPIO6(Battery), GPIO7(Soil/Pyranometer) UART: GPIO43(TX), GPIO44(RX) LED: GPIO2 Agri: GPIO16(SoilTemp), GPIO17(LeafWet), GPIO18(DeepSoil) Solar: GPIO19(PanelTemp/USB_D-), GPIO20(PowerMeter/USB_D+)"
- note removed: "ESP32-S3-WROOM-1-N16R8I INDUSTRIAL Temperature Range: -40C to +85C WiFi: 802.11 b/g/n (2.4GHz, onboard PCB antenna) BLE: v5.0, LE Coded PHY Flash: 16MB (Quad SPI) PSRAM: 8MB (Octal SPI) CPU: Dual Xtensa LX7 @ 240MHz NOTE: Commercial variant (no I suffix) = 0C to +85C only. For outdoor weather stations ALWAYS use the -I variant."
- note removed: "GPIO PIN MAP ───────────────────────────────────────── GPIO0 = BOOT button (active low) GPIO2 = Status LED (green, active high) GPIO4 = Wind Speed (interrupt, 10k pull-up) GPIO5 = Rain Gauge (interrupt, 10k pull-up) GPIO6 = Battery ADC (100k/100k divider) GPIO7 = Industry ADC (soil moisture / pyranometer) GPIO8 = I2C SDA (4.7k pull-up) GPIO9 = I2C SCL (4.7k pull-up) GPIO10 = SPI MOSI (LoRa) GPIO1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"
- note removed: "IMPORTANT: GPIO19/GPIO20 are shared between USB and Solar industry module. Do not use USB while Solar feature is active. For production: use UART for programming."
- title: ESP32-S3 Weather Station — Top Level -> ESP32-S3 Weather Station

Commit message: feat: complete single-MCU migration — remove ESP32-S3, add ATWINC1500/RN4870/W5500/SIM7600
Migrate from dual-MCU (ESP32-S3 + STM32F407) to single-MCU (STM32F407VGT6 only)
with external communication modules:

Firmware changes:
- Rewrite wifi.rs for ATWINC1500 SPI driver, ble.rs for RN4870 UART driver
- Remove all #[cfg(feature = "stm32")] gates — STM32 is now the only target
- Remove bridge protocol (BridgeSync task, USART3 bridge)
- Add PollWifi/PollBle/PollCellular/PollEthernet scheduler tasks
- Update power modes: Sleep(WFI)/Stop/Standby for STM32
- Update OTA for STM32 dual-bank flash swap
- Update config: HEAP 48KB, flash sector 4, new module constants
- Update mode_manager with transport health tracking

Hardware changes:
- Update KiCad schematics (top-level, communication, stm32_scada)
- Update symbol library: replace ESP32-S3 with ATWINC1500/RN4870
- Update BOM: remove ESP32-S3, add ATWINC1500/RN4870/W5500/SIM7600/TPS7A2033
- Update assembly notes for STM32 SWD flashing and new modules

Documentation changes:
- Update all 15 docs and 5 diagram files for single-MCU architecture
- Add v2.0.0 changelog entry
- Replace ESP32 pin numbers with STM32 pin names throughout
- Update build instructions: probe-rs, thumbv7em-none-eabihf target

https://claude.ai/code/session_01XHnfZQ5BbxTCTBMCteQyVe
Other:
- title: ESP32-S3 Weather Station -> STM32F407 Weather Station
Changed lines of the file:
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@@
   (paper "A3")
   (title_block
-    (title "ESP32-S3 Weather Station")
-    (date "2026-02-28")
-    (rev "1.0")
+    (title "STM32F407 Weather Station")
+    (date "2026-03-15")
+    (rev "2.0")
     (company "Weather Station Project")
-    (comment 1 "Top-Level Schematic")
-    (comment 2 "ESP32-S3-WROOM-1 Based")
-    (comment 3 "I2C, SPI, UART, ADC Interfaces")
+    (comment 1 "Top-Level Schematic — Single-MCU Architecture")
+    (comment 2 "STM32F407VGT6 Based — Industrial -40/+105C")
+    (comment 3 "ATWINC1500 WiFi, RN4870 BLE, W5500 Ethernet, SIM7600 Cellular")
     (comment 4 "Hierarchical Design")
   )

Commit message: Add P9E Microsystems branding to board markings
Front silkscreen: P9E (bold), P9E Microsystems Pvt Ltd, www.p9e.in
Back silkscreen: P9E Microsystems Pvt Ltd + www.p9e.in added
Title blocks: company updated to P9E Microsystems Pvt Ltd
Also updated PCB title/rev/date for STM32F407 v2.0

https://claude.ai/code/session_01XHnfZQ5BbxTCTBMCteQyVe
Other:
- company: Weather Station Project -> P9E Microsystems Pvt Ltd
Changed lines of the file:
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@@
     (date "2026-03-15")
     (rev "2.0")
-    (company "Weather Station Project")
+    (company "P9E Microsystems Pvt Ltd")
     (comment 1 "Top-Level Schematic — Single-MCU Architecture")
     (comment 2 "STM32F407VGT6 Based — Industrial -40/+105C")

Commit message: Fix 2: WeatherStation.kicad_sch — remove ESP32-S3, add STM32F407 sub-sheet, fix title/pin annotations
Agent-Logs-Url: https://github.com/ppusapati/weather/sessions/bf78e071-0670-4802-a032-1f4282b37237

Co-authored-by: ppusapati <5749576+ppusapati@users.noreply.github.com>
Parts:
- removed C1: 10uF, Capacitor_SMD:C_0805_2012Metric, symbol Device:C_Polarized
- removed C2: 100nF, Capacitor_SMD:C_0402_1005Metric, symbol Device:C
- removed U1: ESP32-S3-WROOM-1, RF_Module:ESP32-S3-WROOM-1, symbol RF_Module:ESP32-S3-WROOM-1
- SW2: value BOOT -> BOOT0
Other:
- added sheet STM32F407 MCU + SCADA (stm32_scada.kicad_sch)
- note added: "STM32F407 Pin Assignments: I2C1: PB6(SCL), PB7(SDA) SPI1: PA5(SCK), PA6(MISO), PA7(MOSI), PA4(CS-LoRa), PB0(RST), PB1(DIO0) SPI3: PB3(SCK), PB4(MISO), PB5(MOSI) [ATWINC1500 WiFi] USART1: PA9(TX), PA10(RX) [Debug Console] USART3: PB10(TX), PB11(RX) [RN4870 BLE] USART2: PA2(TX), PA3(RX) [MAX3485 RS485] TIM3 CH3/CH4: PB0(Wind), PB1(Rain) ADC1: PC0(Battery), PC1(Soil/Pyranometer) GPIO: PA0(SoilTemp 1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"
- note added: "STM32F407VGT6 Weather Station - Top Level Schematic"
- note removed: "ESP32-S3 Weather Station - Top Level Schematic"
- note removed: "Pin Assignments: I2C: GPIO8(SDA), GPIO9(SCL) SPI: GPIO10(MOSI), GPIO11(MISO), GPIO12(SCK), GPIO13(CS), GPIO14(RST), GPIO15(DIO0) Interrupts: GPIO4(Wind), GPIO5(Rain) ADC: GPIO6(Battery), GPIO7(Soil/Pyranometer) UART: GPIO43(TX), GPIO44(RX) LED: GPIO2 Agri: GPIO16(SoilTemp), GPIO17(LeafWet), GPIO18(DeepSoil) Solar: GPIO19(PanelTemp/USB_D-), GPIO20(PowerMeter/USB_D+)"
